Commit message: Remove the offset

File: resources/ur5/ur5_spherized.urdf (robot description, URDF)
Before this commit: robot ur5_robotiq85, 22 links, 21 joints
Joints:
- joint offset_joint: origin xyz=0.0 0.0 0.9144 rpy=0 0 1.57 -> xyz=0.0 0.0 0.0 rpy=0 0 1.57

Commit message: Add files via upload

File: resources/ur5/ur5_spherized.urdf (robot description, URDF)
Before this commit: robot ur5_robotiq85, 23 links, 22 joints
Links:
- link base_link: geometry collision sphere radius=0.08; visual mesh filename=meshes/ur5/visual/base.dae
- link forearm_link: geometry collision sphere radius=0.04; collision sphere radius=0.04
- link fts_robotside: geometry collision sphere radius=0.04; visual mesh filename=meshes/robotiq_fts300.stl
- link robotiq_85_base_link: geometry collision sphere radius=0.04; collision sphere radius=0.04
- link shoulder_link: geometry collision sphere radius=0.08; visual mesh filename=meshes/ur5/visual/shoulder.dae
- link upper_arm_link: geometry collision sphere radius=0.08; collision sphere radius=0.08
- link wrist_1_link: geometry collision sphere radius=0.04; collision sphere radius=0.04
- link wrist_2_link: geometry collision sphere radius=0.04; collision sphere radius=0.04
- link wrist_3_link: geometry collision sphere radius=0.04; visual mesh filename=meshes/ur5/visual/wrist3.dae
Joints:
- joint offset_joint: origin xyz=0.0 0.0 0.0 rpy=0 0 1.57 -> xyz=0.0 0.0 0.9144 rpy=0 0 1.57
